File: resources/PCB/xmega_motorcontroller/Motorcontroller.brd (EAGLE design)
At the start: 100 x 80 mm, 46 parts, among them IC1 AVR_XMEGA, IC2 REG1118, IC3 L293D

Commit message: xmega pcb updates added to resources
Connections:
- removed net N$21: IC3.15
- removed net N$3: IC1.62
- removed net N$7: IC1.63
- removed net N$9: IC1.64
- net ADC1: now also IC1.62
- net ADC2: now also IC1.63
- net ADC3: now also IC1.64
- net ENCODER_L_1: now also MOTOR_LEFT.3; no longer MOTOR_LEFT.4
- net ENCODER_R_1: now also MOTOR_RIGHT.3; no longer MOTOR_RIGHT.4
- net MOTOR_R_A1: now also IC3.15
Routing:
- net 5V: track 22.5 -> 214.6 mm
- net MOTOR_R_A1: track 0.00 -> 67.9 mm, vias 0 -> 3
- net N$21: track 66.8 -> 0.00 mm, vias 3 -> 0
- net MOTOR_R_POWER_-: track 0.00 -> 46.6 mm
- net PDI_DATA: track 0.00 -> 39.1 mm, vias 0 -> 1
- net MOTOR_L_POWER_+: track 0.00 -> 22.4 mm
- net ENCODER_R_1: track 0.00 -> 21.7 mm, vias 0 -> 1
- net ENCODER_R_1_OUT: track 18.4 -> 38.8 mm
- net MOTOR_R_POWER_+: track 0.00 -> 18.8 mm
- net I2C_SDA: track 0.00 -> 18.7 mm, vias 0 -> 1
- net ENCODER_L_1: track 0.00 -> 17.2 mm
- net VCC: track 276.0 -> 287.2 mm
- net ENCODER_L_1_OUT: track 122.9 -> 133.9 mm
- net LED_1: track 0.00 -> 8.66 mm
- net RESET: track 99.2 -> 104.6 mm
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