File: resources/PCB/xmega_motorcontroller/Motorcontroller.sch (EAGLE design)
At the start: 45 parts, among them IC1 AVR_XMEGA, IC2 REG1118, IC3 L293D

Commit message: xmega pcb updates added to resources
Connections:
- removed net N$21: IC3.4A
- removed net N$3: IC1.PA0
- removed net N$7: IC1.PA1
- removed net N$9: IC1.PA2
- net ADC1: now also IC1.PA0
- net ADC2: now also IC1.PA1
- net ADC3: now also IC1.PA2
- net ENCODER_L_1: now also MOTOR_LEFT.3; no longer MOTOR_LEFT.4
- net ENCODER_R_1: now also MOTOR_RIGHT.3; no longer MOTOR_RIGHT.4
- net MOTOR_R_A1: now also IC3.4A
Other:
- moved on the sheet: ADC#1, ADC#2, ADC#3, MOTOR_LEFT, MOTOR_RIGHT, PDI, Q1, Q2, R1, R10, R12, R13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
