File: resources/PCB/xmeag_motorcontroller_after_updates/Motorcontroller.brd (EAGLE design)
At the start: 100 x 80 mm, 46 parts, among them IC1 AVR_XMEGA, IC2 REG1118, IC3 L293D

Commit message: IR sensor chapter + key words in  i2c chapter
Parts:
- removed C7: (no value), SparkFun-Capacitors:1206
- removed Q1, Q2: (no value), semicon-smd-ipc:SOT23
- removed R10, R12, R13, R3, R4, R8, R9: (no value), SparkFun-Resistors:1206
Connections:
- removed net ENCODER_L_1_OUT: IC1.36, Q1.3, R8.1
- removed net ENCODER_R_1_OUT: IC1.37, Q2.3, R9.1
- removed net N$23: Q1.1, R10.1, R12.1
- removed net N$35: Q2.1, R13.1, R4.1
- new net ENCODER_L_2: IC1.38, MOTOR_LEFT.4
- new net ENCODER_R_2: IC1.39, MOTOR_RIGHT.4
- net 12V: now also C9.2, IC4.IN
- net ENCODER_L_1: now also IC1.36; no longer R12.2
- net ENCODER_R_1: now also IC1.37; no longer R13.2
- net GND: no longer C7.1, Q1.2, Q2.2, R10.2, R4.2
- net RESET: no longer C7.2, R3.1
- net VCC: no longer C9.2, IC4.IN, R3.2, R8.2, R9.2
Routing:
- net ENCODER_L_1_OUT: track 133.9 -> 0.00 mm, vias 2 -> 0
- net ENCODER_L_1: track 17.2 -> 118.8 mm
- net VCC: track 287.2 -> 225.9 mm
- net 12V: track 161.4 -> 214.2 mm
- net ENCODER_R_1_OUT: track 38.8 -> 0.00 mm
- net ENCODER_R_1: track 21.7 -> 0.00 mm, vias 1 -> 0
- net N$23: track 17.6 -> 0.00 mm, vias 2 -> 0
- net GND: track 339.6 -> 328.0 mm
- net N$35: track 11.6 -> 0.00 mm
- net RESET: track 104.6 -> 98.0 mm
