File: resources/PCB/xmeag_motorcontroller_after_updates/Motorcontroller.brd (EAGLE design)
At the start: 100 x 80 mm, 36 parts, among them IC1 AVR_XMEGA, IC2 REG1118, IC3 L293D

Commit message: i2c chapter
Parts:
- R2: value (none) -> 100Ohm
Routing:
- net RESET: track 98.0 -> 89.7 mm
Changed lines of the file:
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@@
 <attribute name="NAME" x="2.54" y="24.765" size="1.27" layer="21" rot="R270"/>
 </element>
-<element name="R2" library="SparkFun-Resistors" package="1206" value="" x="87.63" y="10.16" smashed="yes" rot="R270">
+<element name="R2" library="SparkFun-Resistors" package="1206" value="100Ohm" x="87.63" y="10.16" smashed="yes" rot="R270">
 <attribute name="NAME" x="88.9" y="10.033" size="0.8128" layer="25"/>
 <attribute name="VALUE" x="86.106" y="11.557" size="0.4064" layer="27" rot="R270"/>
@@
 <wire x1="73.66" y1="30.48" x2="67.31" y2="36.83" width="0.8128" layer="16"/>
 <wire x1="67.31" y1="36.83" x2="67.31" y2="39.37" width="0.8128" layer="16"/>
-<wire x1="81.41" y1="71.5115125" x2="90.17" y2="73.66" width="0" layer="19" extent="1-1"/>
-<wire x1="78.74" y1="66.04" x2="76.82120625" y2="71.15700625" width="0" layer="19" extent="1-1"/>
-<wire x1="42.04" y1="57.15" x2="44.45" y2="57.0184875" width="0" layer="19" extent="1-16"/>
-<wire x1="66.04" y1="58.42" x2="60.96" y2="57.15" width="0" layer="19" extent="16-16"/>
-<wire x1="32.76" y1="39.55" x2="39.16" y2="39.55" width="0" layer="19" extent="1-1"/>
-<wire x1="35.56" y1="59.82" x2="42.04" y2="57.15" width="0" layer="19" extent="1-1"/>
-<wire x1="43.36" y1="26.55" x2="43.36" y2="34.55" width="0" layer="19" extent="1-1"/>
-<wire x1="91.44" y1="5.08" x2="87.63" y2="11.56" width="0" layer="19" extent="1-1"/>
-<wire x1="3.81" y1="69.85" x2="11.43" y2="72.39" width="0" layer="19" extent="1-1"/>
-<wire x1="78.74" y1="8.89" x2="86.3584875" y2="12.7" width="0" layer="19" extent="1-1"/>
-<wire x1="15.24" y1="19.05" x2="24.13" y2="29.21" width="0" layer="19" extent="1-1"/>
-<wire x1="10.16" y1="17.78" x2="15.24" y2="19.05" width="0" layer="19" extent="16-16"/>
-<wire x1="5.08" y1="11.43" x2="10.16" y2="7.62" width="0" layer="19" extent="1-1"/>
-<wire x1="8.76" y1="40.64" x2="24.13" y2="29.21" width="0" layer="19" extent="1-1"/>
 </signal>
 <signal name="VCC">
@@
 <wire x1="3.81" y1="35.56" x2="5.08" y2="36.83" width="0.4064" layer="16"/>
 <contactref element="IC1" pad="57"/>
-<wire x1="35.16" y1="39.55" x2="35.16" y2="41.3784875" width="0.4064" layer="1"/>
-<wire x1="35.16" y1="41.3784875" x2="35.25299375" y2="41.60299375" width="0.4064" layer="1" curve="-45"/>
-<wire x1="35.25299375" y1="41.60299375" x2="36.83" y2="43.18" width="0.4064" layer="1"/>
-<wire x1="36.83" y1="43.18" x2="36.83" y2="46.9884875" width="0.4064" layer="1"/>
-<wire x1="36.83" y1="46.9884875" x2="36.92299375" y2="47.21299375" width="0.4064" layer="1" curve="-45"/>
 <wire x1="35.16" y1="37.8315125" x2="35.16" y2="39.55" width="0.4064" layer="1"/>
 <wire x1="39.9288" y1="9.8806" x2="37.33239375" y2="12.47700625" width="0.6096" layer="1"/>
