File: resources/PCB/xmeag_motorcontroller_after_updates/Motorcontroller.sch (EAGLE design)
At the start: 45 parts, among them IC1 AVR_XMEGA, IC2 REG1118, IC3 L293D

Commit message: IR sensor chapter + key words in  i2c chapter
Parts:
- removed C7: (no value), SparkFun-Capacitors:CAP1206
- removed Q1, Q2: (no value), semicon-smd-ipc:NPN-TRANSISTOR_SOT23
- removed R10, R12, R13, R3, R4, R8, R9: (no value), SparkFun-Resistors:RESISTOR1206
Connections:
- removed net ENCODER_L_1_OUT: IC1.PE0, Q1.C, R8.1
- removed net ENCODER_R_1_OUT: IC1.PE1, Q2.C, R9.1
- removed net N$23: Q1.B, R10.1, R12.1
- removed net N$35: Q2.B, R13.1, R4.1
- new net ENCODER_L_2: IC1.PE2, MOTOR_LEFT.4
- new net ENCODER_R_2: IC1.PE3, MOTOR_RIGHT.4
- net 12V: now also C9.2, IC4.IN
- net ENCODER_L_1: now also IC1.PE0; no longer R12.2
- net ENCODER_R_1: now also IC1.PE1; no longer R13.2
- net GND: no longer C7.1, Q1.E, Q2.E, R10.2, R4.2
- net RESET: no longer C7.2, R3.1
- net VCC: no longer C9.2, IC4.IN, R3.2, R8.2, R9.2

Commit message: i2c chapter
Connections:
- removed net N$25: IC3.1A
- removed net N$36: IC3.2A
- removed net N$37: IC3.3-4EN
- removed net N$38: IC3.3A
- removed net N$4: IC3.1-2EN
- net MOTOR_L_A1: now also IC3.1A
- net MOTOR_L_A2: now also IC3.2A
- net MOTOT_R_A2: now also IC3.3A
- net PWM_ML: now also IC3.1-2EN
- net PW_MR: now also IC3.3-4EN
Changed lines of the file:
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@@
 <label x="139.7" y="-25.4" size="1.27" layer="95" rot="R180" xref="yes"/>
+</segment>
+<segment>
+<pinref part="IC3" gate="G$1" pin="1-2EN"/>
+<wire x1="233.68" y1="5.08" x2="220.98" y2="5.08" width="0.1524" layer="91"/>
 </segment>
 </net>
@@
 <label x="139.7" y="-27.94" size="1.27" layer="95" rot="R180" xref="yes"/>
 </segment>
+<segment>
+<pinref part="IC3" gate="G$1" pin="3-4EN"/>
+<wire x1="264.16" y1="-30.48" x2="279.4" y2="-30.48" width="0.1524" layer="91"/>
+</segment>
 </net>
 <net name="MOTOR_L_A1" class="0">
@@
 <label x="144.78" y="-30.48" size="1.27" layer="95" rot="R180" xref="yes"/>
 </segment>
+<segment>
+<pinref part="IC3" gate="G$1" pin="1A"/>
+<wire x1="233.68" y1="0" x2="220.98" y2="0" width="0.1524" layer="91"/>
+</segment>
 </net>
 <net name="MOTOR_L_A2" class="0">
@@
 <label x="220.98" y="-25.4" size="1.778" layer="95" rot="R180" xref="yes"/>
 <label x="144.78" y="-33.02" size="1.27" layer="95" rot="R180" xref="yes"/>
+</segment>
+<segment>
+<pinref part="IC3" gate="G$1" pin="2A"/>
+<wire x1="233.68" y1="-25.4" x2="220.98" y2="-25.4" width="0.1524" layer="91"/>
 </segment>
 </net>
@@
 <label x="144.78" y="-38.1" size="1.27" layer="95" rot="R180" xref="yes"/>
 </segment>
-</net>
-<net name="N$25" class="0">
 <segment>
-<pinref part="IC3" gate="G$1" pin="1A"/>
-<wire x1="233.68" y1="0" x2="220.98" y2="0" width="0.1524" layer="91"/>
+<pinref part="IC3" gate="G$1" pin="3A"/>
+<wire x1="264.16" y1="-25.4" x2="279.4" y2="-25.4" width="0.1524" layer="91"/>
 </segment>
 </net>
@@
 <wire x1="205.74" y1="-83.82" x2="205.74" y2="-81.28" width="0.1524" layer="91"/>
 <wire x1="205.74" y1="-83.82" x2="205.74" y2="-76.2" width="0.1524" layer="91"/>
-</segment>
-</net>
-<net name="N$36" class="0">
-<segment>
-<pinref part="IC3" gate="G$1" pin="2A"/>
-<wire x1="233.68" y1="-25.4" x2="220.98" y2="-25.4" width="0.1524" layer="91"/>
-</segment>
-</net>
-<net name="N$37" class="0">
-<segment>
-<pinref part="IC3" gate="G$1" pin="3-4EN"/>
-<wire x1="264.16" y1="-30.48" x2="279.4" y2="-30.48" width="0.1524" layer="91"/>
-</segment>
-</net>
-<net name="N$38" class="0">
-<segment>
-<pinref part="IC3" gate="G$1" pin="3A"/>
-<wire x1="264.16" y1="-25.4" x2="279.4" y2="-25.4" width="0.1524" layer="91"/>
 </segment>
 </net>
@@
 </segment>
 </net>
-<net name="N$4" class="0">
-<segment>
-<pinref part="IC3" gate="G$1" pin="1-2EN"/>
-<wire x1="233.68" y1="5.08" x2="220.98" y2="5.08" width="0.1524" layer="91"/>
-</segment>
-</net>

Commit message: i2c chapter
Parts:
- R2: value (none) -> 100Ohm
Other:
- moved on the sheet: C1, C10, C2, C8, C9, D1, D2, D3, I2C#1, I2C#2, IC2, IC3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
