File: resources/PCB/Eyebot_powerdist/Eyebot_powerdist.brd (EAGLE design)
At the start: 100 x 80 mm, 33 parts, among them IC3 MCP23016SO, K1 62000211622, K2 62000211622, K3 62000211622, K4 62000211622, K5 62000211622, K6 62000211622, K7 61201021621, Q1 2N2222, Q2 2N2222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

Commit message: i2c chapter
Connections:
- net N$16 renamed LED5
- net N$29 renamed BUZZER
- net N$34 renamed SCL
- net N$35 renamed SDA
- net N$38 renamed LED7
- net N$42 renamed LED3
- net N$44 renamed LED1
- removed net N$12 (its old number): K7.6, R21.2
- removed net N$14 (its old number): K7.8, R23.2
- removed net N$37: IC3.28, R23.1
- removed net N$39: IC3.26, R21.1
- removed net N$41: IC3.24, R19.1
- removed net N$43: IC3.22, R17.1
- new net LED2: IC3.22, R17.2
- new net LED4: IC3.24, R19.2
- new net LED6: IC3.26, R21.2
- new net LED8: IC3.28, R23.2
- new net N$4: K7.2, R17.1
- new net N$9: K7.6, R21.1
- net N$10: now also K7.8, R23.1; no longer K7.4, R19.2
- net N$6: now also K7.4, R19.1; no longer K7.2, R17.2
Routing:
- net LED1: track 45.5 -> 0.00 mm, vias 1 -> 0
- net SDA: track 37.7 -> 0.00 mm, vias 1 -> 0
- net N$43: track 28.0 -> 0.00 mm, vias 1 -> 0
- net N$6: track 23.8 -> 0.00 mm
- net LED3: track 23.1 -> 0.00 mm
- net N$37: track 19.0 -> 0.00 mm, vias 1 -> 0
- net N$16: track 18.4 -> 0.00 mm
- net LED7: track 17.7 -> 0.00 mm, vias 1 -> 0
- net N$14 (its old number): track 17.7 -> 0.00 mm
- net N$41: track 17.5 -> 0.00 mm, vias 1 -> 0
- net LED5: track 17.0 -> 0.00 mm, vias 1 -> 0
- net N$10: track 16.9 -> 0.00 mm
- net N$39: track 15.4 -> 0.00 mm, vias 1 -> 0
- net N$12 (its old number): track 13.8 -> 0.00 mm
- net N$14: track 12.3 -> 0.00 mm
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
Commit message: Simulink files
Parts:
- C1: value (none) -> 0.1u
- C2: value (none) -> 0.33u
- C3, C4: value (none) -> 4.7u
- R15: value (none) -> 4k
- turned R17 to 270 degrees
- turned R19 to 270 degrees
- turned R21 to 270 degrees
- turned R23 to 270 degrees
Routing:
- net LED8: track 0.00 -> 15.1 mm
Changed lines of the file:
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@@
 <elements>
 <element name="IC1" library="SparkFun-PowerIC" package="TO-220-ALT" value="" x="74.93" y="58.42"/>
-<element name="C1" library="SparkFun-Capacitors" package="AXIAL-5MM" value="" x="85.09" y="62.23" rot="R90"/>
-<element name="C2" library="SparkFun-Capacitors" package="CAP-PTH-SMALL" value="" x="67.31" y="59.69" rot="R90"/>
+<element name="C1" library="SparkFun-Capacitors" package="AXIAL-5MM" value="0.1u" x="85.09" y="62.23" rot="R90"/>
+<element name="C2" library="SparkFun-Capacitors" package="CAP-PTH-SMALL" value="0.33u" x="67.31" y="59.69" rot="R90"/>
 <element name="Q1" library="transistor-npn" package="TO18" value="2N2222" x="13.97" y="34.29"/>
 <element name="Q2" library="transistor-npn" package="TO18" value="2N2222" x="13.97" y="25.4"/>
@@
 <element name="K5" library="Wuerth_Elektronik_eiCan_09_Wire_to_Board_Connectors" package="62000211622" value="62000211622" x="96.52" y="41.91" rot="R270"/>
 <element name="IC2" library="dan-vreg" package="SOT223-3L" value="" x="59.69" y="72.39"/>
-<element name="C3" library="SparkFun-Capacitors" package="1206" value="" x="57.15" y="66.04" rot="R180"/>
-<element name="C4" library="SparkFun-Capacitors" package="1206" value="" x="62.23" y="64.77" rot="R270"/>
+<element name="C3" library="SparkFun-Capacitors" package="1206" value="4.7u" x="57.15" y="66.04" rot="R180"/>
+<element name="C4" library="SparkFun-Capacitors" package="1206" value="4.7u" x="62.23" y="64.77" rot="R270"/>
 <element name="K6" library="Wuerth_Elektronik_eiCan_09_Wire_to_Board_Connectors" package="62000211622" value="62000211622" x="22.86" y="5.08"/>
 <element name="K7" library="Wuerth_Elektronik_eiCan_05_Box_Header_IDC_Connectors_1_2" package="61201021621" value="61201021621" x="35.56" y="72.39"/>
@@
 <attribute name="OC_FARNELL" value="unknown" x="96.52" y="3.81" size="1.778" layer="27" display="off"/>
 </element>
-<element name="R15" library="resistor" package="0309/10" value="" x="13.97" y="44.45"/>
+<element name="R15" library="resistor" package="0309/10" value="4k" x="13.97" y="44.45"/>
 <element name="IC3" library="microchip2" package="SO-28W" value="MCP23016SO" x="31.75" y="36.83" rot="R270"/>
 <element name="R16" library="resistor" package="0309/10" value="" x="20.32" y="55.88" rot="R90"/>
-<element name="R17" library="resistor" package="0309/10" value="" x="15.24" y="55.88" rot="R90"/>
+<element name="R17" library="resistor" package="0309/10" value="" x="15.24" y="55.88" rot="R270"/>
 <element name="R18" library="resistor" package="0309/10" value="" x="30.48" y="55.88" rot="R90"/>
-<element name="R19" library="resistor" package="0309/10" value="" x="25.4" y="55.88" rot="R90"/>
+<element name="R19" library="resistor" package="0309/10" value="" x="25.4" y="55.88" rot="R270"/>
 <element name="R20" library="resistor" package="0309/10" value="" x="35.56" y="55.88" rot="R90"/>
-<element name="R21" library="resistor" package="0309/10" value="" x="40.64" y="55.88" rot="R90"/>
+<element name="R21" library="resistor" package="0309/10" value="" x="40.64" y="55.88" rot="R270"/>
 <element name="R22" library="resistor" package="0309/10" value="" x="45.72" y="55.88" rot="R90"/>
-<element name="R23" library="resistor" package="0309/10" value="" x="50.8" y="55.88" rot="R90"/>
+<element name="R23" library="resistor" package="0309/10" value="" x="50.8" y="55.88" rot="R270"/>
 </elements>
 <signals>
@@
 <contactref element="K7" pad="2"/>
 <contactref element="R17" pad="1"/>
-<wire x1="15.24" y1="50.8" x2="33.02" y2="73.66" width="0" layer="19" extent="1-1"/>
+<wire x1="15.24" y1="60.96" x2="33.02" y2="73.66" width="0" layer="19" extent="1-1"/>
 </signal>
 <signal name="N$6">
 <contactref element="K7" pad="4"/>
 <contactref element="R19" pad="1"/>
-<wire x1="25.4" y1="50.8" x2="35.56" y2="73.66" width="0" layer="19" extent="1-1"/>
+<wire x1="25.4" y1="60.96" x2="35.56" y2="73.66" width="0" layer="19" extent="1-1"/>
 </signal>
 <signal name="N$9">
 <contactref element="K7" pad="6"/>
 <contactref element="R21" pad="1"/>
-<wire x1="40.64" y1="50.8" x2="38.1" y2="73.66" width="0" layer="19" extent="1-1"/>
+<wire x1="40.64" y1="60.96" x2="38.1" y2="73.66" width="0" layer="19" extent="1-1"/>
 </signal>
 <signal name="N$10">
 <contactref element="K7" pad="8"/>
 <contactref element="R23" pad="1"/>
-<wire x1="50.8" y1="50.8" x2="40.64" y2="73.66" width="0" layer="19" extent="1-1"/>
+<wire x1="50.8" y1="60.96" x2="40.64" y2="73.66" width="0" layer="19" extent="1-1"/>
 </signal>
 <signal name="N$12">
@@
 <contactref element="IC3" pad="22"/>
 <contactref element="R17" pad="2"/>
-<wire x1="36.703" y1="36.83" x2="15.24" y2="60.96" width="0" layer="19" extent="1-1"/>
+<wire x1="36.703" y1="36.83" x2="15.24" y2="50.8" width="0" layer="19" extent="1-1"/>
 </signal>
 <signal name="LED3">
@@
 <contactref element="IC3" pad="24"/>
 <contactref element="R19" pad="2"/>
-<wire x1="36.703" y1="39.37" x2="25.4" y2="60.96" width="0" layer="19" extent="1-1"/>
+<wire x1="36.703" y1="39.37" x2="25.4" y2="50.8" width="0" layer="19" extent="1-1"/>
 </signal>
 <signal name="LED5">
@@
 <contactref element="IC3" pad="26"/>
 <contactref element="R21" pad="2"/>
-<wire x1="36.703" y1="41.91" x2="40.64" y2="60.96" width="0" layer="19" extent="1-1"/>
+<wire x1="36.703" y1="41.91" x2="40.64" y2="50.8" width="0" layer="19" extent="1-1"/>
 </signal>
 <signal name="LED7">
@@
 <contactref element="IC3" pad="28"/>
 <contactref element="R23" pad="2"/>
-<wire x1="36.703" y1="44.45" x2="50.8" y2="60.96" width="0" layer="19" extent="1-1"/>
+<wire x1="36.703" y1="44.45" x2="36.83" y2="44.45" width="0.4064" layer="1"/>
+<wire x1="36.83" y1="44.45" x2="39.37" y2="46.99" width="0.4064" layer="1"/>
+<wire x1="39.37" y1="46.99" x2="50.8" y2="46.99" width="0.4064" layer="1"/>
+<wire x1="50.8" y1="46.99" x2="50.8" y2="50.8" width="0" layer="19" extent="1-16"/>
 </signal>
 <signal name="BUZZER">
