File: resources/PCB/Eyebot_powerdist/Eyebot_powerdist.sch (EAGLE design)
At the start: 33 parts, among them IC3 MCP23016SO, K1 62000211622, K2 62000211622, K3 62000211622, K4 62000211622, K5 62000211622, K6 62000211622, K7 61201021621, Q1 2N2222, Q2 2N2222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

Commit message: i2c chapter
Connections:
- net N$16 renamed LED5
- net N$29 renamed BUZZER
- net N$34 renamed SCL
- net N$35 renamed SDA
- net N$38 renamed LED7
- net N$42 renamed LED3
- net N$44 renamed LED1
- removed net N$12 (its old number): K7.6, R21.2
- removed net N$14 (its old number): K7.8, R23.2
- removed net N$37: IC3.GP0.7, R23.1
- removed net N$39: IC3.GP0.5, R21.1
- removed net N$41: IC3.GP0.3, R19.1
- removed net N$43: IC3.GP0.1, R17.1
- new net LED2: IC3.GP0.1, R17.2
- new net LED4: IC3.GP0.3, R19.2
- new net LED6: IC3.GP0.5, R21.2
- new net LED8: IC3.GP0.7, R23.2
- new net N$4: K7.2, R17.1
- new net N$9: K7.6, R21.1
- net N$10: now also K7.8, R23.1; no longer K7.4, R19.2
- net N$6: now also K7.4, R19.1; no longer K7.2, R17.2
Other:
- note added: "8 x 100 ohm"
- moved on the sheet: C1, C2, C3, C4, IC1, IC2, K1, K2, K3, K4, K5, K6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

Commit message: Simulink files
Parts:
- C1: value (none) -> 0.1u
- C2: value (none) -> 0.33u
- C3, C4: value (none) -> 4.7u
- R15: value (none) -> 4k
Changed lines of the file:
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@@
 <parts>
 <part name="IC1" library="SparkFun-PowerIC" deviceset="V_REG_78XX" device="-TO-220"/>
-<part name="C1" library="SparkFun-Capacitors" deviceset="CAP" device="_"/>
-<part name="C2" library="SparkFun-Capacitors" deviceset="CAP" device="PTH"/>
+<part name="C1" library="SparkFun-Capacitors" deviceset="CAP" device="_" value="0.1u"/>
+<part name="C2" library="SparkFun-Capacitors" deviceset="CAP" device="PTH" value="0.33u"/>
 <part name="GND1" library="supply1" deviceset="GND" device=""/>
 <part name="Q1" library="transistor-npn" deviceset="2N2222*" device=""/>
@@
 <part name="K5" library="Wuerth_Elektronik_eiCan_09_Wire_to_Board_Connectors" deviceset="62000211622" device=""/>
 <part name="IC2" library="dan-vreg" deviceset="LDO1117" device="-SOT223"/>
-<part name="C3" library="SparkFun-Capacitors" deviceset="CAP" device="1206"/>
-<part name="C4" library="SparkFun-Capacitors" deviceset="CAP" device="1206"/>
+<part name="C3" library="SparkFun-Capacitors" deviceset="CAP" device="1206" value="4.7u"/>
+<part name="C4" library="SparkFun-Capacitors" deviceset="CAP" device="1206" value="4.7u"/>
 <part name="GND6" library="supply1" deviceset="GND" device=""/>
 <part name="K6" library="Wuerth_Elektronik_eiCan_09_Wire_to_Board_Connectors" deviceset="62000211622" device=""/>
@@
 <part name="Q3" library="transistor-npn" deviceset="2N2222*" device=""/>
 <part name="SG1" library="buzzer" deviceset="F/CM12P" device=""/>
-<part name="R15" library="resistor" deviceset="R-US_" device="0309/10"/>
+<part name="R15" library="resistor" deviceset="R-US_" device="0309/10" value="4k"/>
 <part name="GND8" library="supply1" deviceset="GND" device=""/>
 <part name="IC3" library="microchip2" deviceset="MCP23016" device="SO"/>
